File: mouse_v4.sch (EAGLE design)
At the start: 71 parts

Commit message: Changed IR LED Resistors
Switched voltage from 5V to 3.3V for IR LEDs, and changed resistor values accordingly
Parts:
- R_IR-FL1, R_IR-FR1, R_IR-L1, R_IR-R1: value 51 -> 15
Connections:
- net 3V3: now also C_IR-FL1.1, C_IR-FL2.1, C_IR-FR1.1, C_IR-FR2.1, C_IR-L1.1, C_IR-L2.1, C_IR-R1.1, C_IR-R2.1, IR_FL.+, IR_FR.+, IR_L.+, IR_R.+
- net 5V: no longer C_IR-FL1.1, C_IR-FL2.1, C_IR-FR1.1, C_IR-FR2.1, C_IR-L1.1, C_IR-L2.1, C_IR-R1.1, C_IR-R2.1, IR_FL.+, IR_FR.+, IR_L.+, IR_R.+
