File: mouse_v6.sch (EAGLE design)
At the start: 71 parts, among them U2 DRV8835DSSR

Commit message: updates I never pushed
Parts:
- removed C_5VREG1: 0.33uF, SparkFun:CAP0603-CAP
- removed C_5VREG2: 0.1uF, SparkFun:CAP0603-CAP
- removed REG_5V: MC7805, MC33269:MC7805
- removed U2: DRV8835DSSR, DRV8835:DRV8835DSSR
- added U$9: DRV8835, DRV8835:DRV8835
- R_IR-FL1, R_IR-FR1, R_IR-L1, R_IR-R1: value 51 -> 15
Connections:
- removed net 5V: C_3V3REG2.2, C_5VREG2.1, C_HB-MOTOR.2, C_IR-FL1.1, C_IR-FL2.1, C_IR-FR1.1, C_IR-FR2.1, C_IR-L1.1, C_IR-L2.1, C_IR-R1.1, C_IR-R2.1, IR_FL.+, IR_FR.+, IR_L.+, IR_R.+, REG_3V3.VIN, REG_5V.VOUT, U2.VM
- net 3V3: now also C_HB-MOTOR.2, C_IR-FL1.1, C_IR-FL2.1, C_IR-FR1.1, C_IR-FR2.1, C_IR-L1.1, C_IR-L2.1, C_IR-R1.1, C_IR-R2.1, IR_FL.+, IR_FR.+, IR_L.+, IR_R.+, U$9.VM
- net BAT: now also C_3V3REG2.2, REG_3V3.VIN, U$9.VCC; no longer C_5VREG1.1, REG_5V.VIN, U2.VCC
- net GND: no longer C_5VREG1.2, C_5VREG2.2, REG_5V.GND
- net HB_B1: now also U$9.AIN2/AENBL; no longer U2.AIN2/AENBL
- net HB_B2: now also U$9.BIN2/BENBL; no longer U2.BIN2/BENBL
- net HB_F1: now also U$9.AIN1/APHASE; no longer U2.AIN1/APHASE
- net HB_F2: now also U$9.BIN1/BPHASE; no longer U2.BIN1/BPHASE
- net HB_MODE: now also U$9.MODE; no longer U2.MODE
- net LED2: now also U$1.PC6; no longer U$1.PC14
- net MGND: now also U$9.EPAD, U$9.GND; no longer U2.EPAD, U2.GND
- net M_B1: now also U$9.AOUT2; no longer U2.AOUT2
- net M_B2: now also U$9.BOUT2; no longer U2.BOUT2
- net M_F1: now also U$9.AOUT1; no longer U2.AOUT1
- net M_F2: now also U$9.BOUT1; no longer U2.BOUT1
Other:
- note removed: "MC7805 - 5V Regulator"
- note removed: "RX"
- note removed: "TX"
- moved on the sheet: C_3V3REG1, C_3V3REG2, REG_3V3
