File: mouse_v6.brd (EAGLE design)
At the start: 100 x 65 mm, 71 parts

Commit message: updates I never pushed
Parts:
- removed C_5VREG1: 0.33uF, SparkFun:0603-CAP
- removed C_5VREG2: 0.1uF, SparkFun:0603-CAP
- removed REG_5V: MC7805, MC33269:TO-252-3
- R_IR-FL1, R_IR-FR1, R_IR-L1, R_IR-R1: value 51 -> 15
- moved LED2 78.6 mm to (70.3, 61.6), turned to 0 degrees
- moved R_LED2 74.0 mm to (70.3, 58.5), turned to 270 degrees
- moved LED1 50.0 mm to (69.6, 3.35)
- moved R_LED1 47.8 mm to (67.5, 5.67), turned to 180 degrees
- moved U$8 36.9 mm to (5.34, 62.3), flipped to the bottom
- moved R_IR-R3 11.3 mm to (81.3, 8.08), turned to 0 degrees
- moved R_IR-L3 10.3 mm to (91.9, 43.5)
- moved C_IR-FL1 9.00 mm to (79.0, 49.9)
- moved C_IR-FL2 9.00 mm to (79.0, 47.2)
- moved C_IR-FR1 9.00 mm to (78.4, 20.9)
- moved C_IR-FR2 9.00 mm to (78.4, 18.2)
- moved IR_FL 9.00 mm to (82.5, 47.3)
- moved IR_FR 9.00 mm to (82.5, 17.5)
- moved R_IR-FL1 9.00 mm to (79.1, 44.8)
- moved R_IR-FL2 9.00 mm to (75.8, 48.5)
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Connections:
- removed net 5V: C_3V3REG2.2, C_5VREG2.1, C_HB-MOTOR.2, C_IR-FL1.1, C_IR-FL2.1, C_IR-FR1.1, C_IR-FR2.1, C_IR-L1.1, C_IR-L2.1, C_IR-R1.1, C_IR-R2.1, IR_FL.+, IR_FR.+, IR_L.+, IR_R.+, REG_3V3.3, REG_5V.4, U$9.1
- net 3V3: now also C_HB-MOTOR.2, C_IR-FL1.1, C_IR-FL2.1, C_IR-FR1.1, C_IR-FR2.1, C_IR-L1.1, C_IR-L2.1, C_IR-R1.1, C_IR-R2.1, IR_FL.+, IR_FR.+, IR_L.+, IR_R.+, U$9.1
- net BAT: now also C_3V3REG2.2, REG_3V3.3; no longer C_5VREG1.1, REG_5V.3
- net GND: no longer C_5VREG1.2, C_5VREG2.2, REG_5V.1
- net LED2: now also U$1.PC6; no longer U$1.PC14
Routing:
- net GND: track 510.7 -> 131.4 mm, vias 13 -> 19
- net 3V3: track 359.5 -> 45.9 mm, vias 8 -> 2
- net 5V: track 245.0 -> 0.00 mm, vias 4 -> 0
- net MGND: track 15.8 -> 59.7 mm, vias 0 -> 5
- net LED2: track 58.3 -> 21.1 mm, vias 0 -> 2
- net LED1: track 56.8 -> 23.9 mm, vias 0 -> 2
- net M_F1: track 5.58 -> 23.9 mm
- net M_F2: track 24.1 -> 6.12 mm
- net NRST: track 128.8 -> 111.6 mm, vias 0 -> 4
- net BAT: track 62.5 -> 47.8 mm, vias 3 -> 2
- net M_B2: track 20.9 -> 8.30 mm
- net ENC_B2: track 27.6 -> 15.7 mm, vias 0 -> 2
- net M_B1: track 9.69 -> 21.4 mm
- net REC_L: track 40.1 -> 33.3 mm, vias 2 -> 0
- net EMIT_FR: track 20.8 -> 14.5 mm, vias 0 -> 2
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- added copper zone on layer 1, net 3V3
Other:
- board size 100 x 65 mm -> 98 x 65 mm

Commit message: pcb width
Parts:
- removed NRST_SWITCH: (no value), switch-omron:B3F-10XX
- removed S1: (no value), SparkFun:SWITCH-SPDT_KIT
- removed S2: (no value), switch-dil:DS-01
- added U$10, U$11: SMD_SWITCH, switches:SMD_SWITCH
- added U$12: SMD_BUTTON, switches:SMD_BUTTON
- moved R_LED2 23.9 mm to (63.7, 81.5), turned to 90 degrees
- moved LED2 21.9 mm to (61.3, 81.7)
- moved PIN_HEADERS 18.0 mm to (63.0, 74.5)
- moved C_IR-R1 10.0 mm to (87.8, 22.3)
- moved C_3V3REG1 10.0 mm to (15.4, 52.9)
- moved C_3V3REG2 10.0 mm to (22.7, 57.7)
- moved C_G1 10.0 mm to (85.0, 39.0)
- moved C_G2 10.0 mm to (85.0, 41.2)
- moved C_HB-BAT 10.0 mm to (26.1, 44.2)
- moved C_HB-MOTOR 10.0 mm to (26.1, 40.9)
- moved C_IR-FL1 10.0 mm to (79.0, 59.9)
- moved C_IR-FL2 10.0 mm to (79.0, 57.2)
- moved C_IR-FR1 10.0 mm to (78.4, 30.9)
- moved C_IR-FR2 10.0 mm to (78.4, 28.2)
- moved C_IR-L1 10.0 mm to (89.4, 63.9)
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Connections:
- net 3V3: now also U$11.1; no longer S2.2
- net BAT: now also U$10.2; no longer S1.2
- net BOOT0: now also U$11.2; no longer S2.1
- net GND: now also U$12.3, U$12.4; no longer NRST_SWITCH.1
- net N$6: now also U$10.1; no longer S1.3
- net NRST: now also U$12.1, U$12.2; no longer NRST_SWITCH.3
Routing:
- net LED2: track 21.1 -> 37.4 mm
- net GND: track 131.4 -> 141.7 mm, vias 19 -> 20
- net NRST: track 111.6 -> 120.5 mm
- net BOOT0: track 66.3 -> 74.8 mm, vias 5 -> 6
- net SWDIO: track 20.3 -> 28.4 mm
- net TX: track 18.2 -> 26.2 mm
- net RX: track 17.4 -> 25.4 mm
- net SWCLK: track 38.4 -> 45.8 mm
- net LED1: track 23.9 -> 29.5 mm
- net N$6: track 6.22 -> 10.3 mm
- net BAT: track 47.8 -> 50.7 mm
- net N$10: track 1.53 -> 2.44 mm
- net MGND: track 59.7 -> 60.0 mm, vias 5 -> 6
Other:
- board size 98 x 65 mm -> 98 x 85 mm
